File: SDTV2CSI.kicad_sch (KiCad schematic)
At the start: 101 parts, among them J1 Conn_Coaxial, J2 Conn_Coaxial, J3 SFW15R-1STE1LF, J4 Conn_Coaxial, J5 Conn_Coaxial, J6 Conn_Coaxial, J7 Conn_Coaxial, J8 Conn_Coaxial, J9 Conn_Coaxial, P1 Pi Zero, P2 TMJ19911ADNL, U1 ADV7280AWBCPZ-M, U2 TLV75718, U3 XR22800IL32TR-F, U4 MP8007GV-Z, Y1 28.63636MHz

Commit message: updating for GitHub
Parts:
- removed C28, C29: 0.01μF, Capacitor_SMD:C_0402_1005Metric, symbol Device:C_Small
- removed D1: 30VZD, Diode_SMD:D_SOD-123F, symbol Device:D_Zener
- removed D2: BAT46W, Diode_SMD:D_SOD-123, symbol Device:D_Schottky
- removed D3: D_Schottky, Diode_SMD:D_SMA, symbol Device:D_Schottky
- removed D4: BR, Diode_SMD:Diode_Bridge_Diotec_SO-DIL-Slim, symbol Diode_Bridge:DF01S1
- removed D5: SBR8U60P5-13, symbol Device:D_Small
- removed F1, F2, F3, F4, F5: LC(PI), AU:NFE31PT101C1E9L_MUR, symbol AU:NFE31PT101C1E9L
- removed FB1, FB2: 30m, Inductor_SMD:L_0603_1608Metric, symbol Device:FerriteBead_Small
- removed J1, J2, J4, J5, J6, J7, J8, J9: Conn_Coaxial, Connector_Coaxial:SMA_Amphenol_901-144_Vertical, symbol Connector:Conn_Coaxial
- removed L1: L_Small, symbol Device:L_Small
- removed P2: TMJ19911ADNL, AU:7498210220A, symbol AU:TMJ19911ADNL
- removed R22: 576, Resistor_SMD:R_0402_1005Metric, symbol Device:R_Small
- removed TR1: CX9628, AU:SMT_29-ALD_COC, symbol AU:CX9628
- removed U3: XR22800IL32TR-F, AU:QFN-32-1EP_5x5mm_P0.5mm_EP3.8x3.8mm, symbol AU:XR22800IL32TR-F
- removed U4: MP8007GV-Z, AU:QFN50P500X400X100-29N, symbol AU:MP8007GV-Z
- added C? (x4): 0.1μF, AU:R_0201_0603Metric, symbol Device:C_Small
- added D18: LED_Dual_AAK, Package_TO_SOT_SMD:SOT-23, symbol Device:LED_Dual_AAK
- added F1, F2, F3, F4, F5: LC(Pi), AU:MEM1608P25R0T001, symbol AU:MEM1608P25R0T001
- added J10, J11: Conn_02x08_Odd_Even, symbol Connector_Generic:Conn_02x08_Odd_Even
- added Q?: PFET, AU:CSD23280F3, symbol AU:CSD23280F3
- added R? (x5): 4.7k, Resistor_SMD:R_0201_0603Metric, symbol Device:R_Small
- added U3: TCA9555RGER, Package_DFN_QFN:VQFN-24-1EP_4x4mm_P0.5mm_EP2.45x2.45mm, symbol Interface_Expansion:TCA9555RGER
- added U4, U5, U6, U7: TS3DS10224RUK, Package_DFN_QFN:WQFN-20-1EP_3x3mm_P0.4mm_EP1.7x1.7mm, symbol Analog_Switch:TS3DS10224RUK
- D1, D2, D3, D4: renamed from D?; symbol Device:D_TVS -> Device:D_Zener_Small
- D10, D11, D12, D13, D14, D15, D16, D17: renamed from D?; value D_TVS -> TVS; symbol Device:D_TVS -> Device:D_Zener_Small
- D5, D6, D7, D8, D9: renamed from D?; value D_TVS -> 3VWM; symbol Device:D_TVS -> Device:D_Zener_Small
- R18: value 3k -> 560; footprint Resistor_SMD:R_0201_0603Metric -> AU:R_0201_0603Metric; Alt PN (none) -> CRCW0201560RFKED; MPN PFR03S-302-FNH -> ERA-1AEB561C; Manufacturer Delta Electronics/Cyntec -> Panasonic Electronic Components; Power 1/20W -> (none)
- R19: value 7.5k -> 220; footprint Resistor_SMD:R_0402_1005Metric -> AU:R_0201_0603Metric; Alt PN CR0402-FX-7501GLF -> RC0201FR-07220RL; MPN WR04X7501FTL -> WR02X2200FAL; Tolerance (none) -> 1%
- R8: value 24.9kΩ -> 560; footprint Resistor_SMD:R_0402_1005Metric -> AU:R_0201_0603Metric; Alt PN (none) -> CRCW0201560RFKED; MPN CR0402-FX-2492GLF -> ERA-1AEB561C; Manufacturer Bourns Inc. -> Panasonic Electronic Components; Tolerance (none) -> 1%
- renumbered J3 to J9
Connections:
- net VDD is gone; now on an unnamed net: R8.1
- net +1V8: now also F2.1, F3.1, F4.1, F5.1
- net +3V3: now also D5.1 (K), C?.1, C?.1, C?.1, C?.1, F1.1, Q?.2, R?.2, R?.2, R?.2, R?.2, U4.13 (VCC), U5.13 (VCC), U6.13 (VCC), U7.13 (VCC); no longer C22.2, J9.1, U2.1 (IN), U2.3 (EN)
- net AVDD: now also F5.3
- net CD0+: now also D3.1 (K)
- net CD0-: now also D4.1 (K)
- net CLK+: now also D1.1 (K)
- net CLK-: now also D2.1 (K)
- net CSCL: now also D7.1 (K), U3.19 (SCL)
- net CSDA: now also D6.1 (K), U3.20 (SDA)
- net DVDD: now also F3.3
- net DVDDIO: now also F1.3
- net GND: now also D1.2 (A), D10.2 (A), D11.2 (A), D12.2 (A), D13.2 (A), D14.2 (A), D15.2 (A), D16.2 (A), D17.2 (A), D2.2 (A), D3.2 (A), D4.2 (A), D5.2 (A), D6.2 (A), D7.2 (A), D8.2 (A), D9.2 (A), C?.2, C?.2, C?.2, C?.2, D18.3 (K), F1.2_4, F2.2_4, F3.2_4, F4.2_4, F5.2_4, J10.10 (Pin_10), J10.12 (Pin_12), J10.14 (Pin_14), J10.16 (Pin_16), J10.2 (Pin_2), J10.4 (Pin_4), J10.6 (Pin_6), J10.8 (Pin_8), U3.18 (A0), U3.23 (A1), U3.24 (A2), U3.25 (EPAD), U3.9 (GND), U4.11 (SBO), U4.12 (SBI), U4.15 (SAO), U4.5 (GND), U5.11 (SBO), U5.12 (SBI), U5.15 (SAO), U5.5 (GND), U6.11 (SBO), U6.12 (SBI), U6.15 (SAO), U6.5 (GND), U7.11 (SBO), U7.12 (SBI), U7.15 (SAO), U7.5 (GND)
- net LED_EN: now also D8.1 (K), R18.2, R8.2; no longer J9.4
- net MVDD: now also F2.3
- net PVDD: now also F4.3
- net PWR_EN: now also D9.1 (K), R19.2
- net video_in1: now also D10.1 (K), J10.1 (Pin_1)
- net video_in2: now also D11.1 (K), J10.3 (Pin_3)
- net video_in3: now also D12.1 (K), J10.5 (Pin_5)
- net video_in4: now also D13.1 (K), J10.7 (Pin_7)
- net video_in5: now also D14.1 (K), J10.9 (Pin_9)
- net video_in6: now also D15.1 (K), J10.11 (Pin_11)
- net video_in7: now also D16.1 (K), J10.13 (Pin_13)
- net video_in8: now also D17.1 (K), J10.15 (Pin_15)
- net at R19.1: now also D18.2 (A2); no longer R18.2
- net at R18.1: now also D18.1 (A1)
- new net: R?.1, U6.14 (SAI)
- new net: R?.1, U5.14 (SAI)
- new net: R?.1, U7.14 (SAI)
- new net: R?.2, U3.22 (~{INT})
- new net: R?.1, U4.14 (SAI)
- new net 3V3: C22.2, J9.1, Q?.3, R?.1, U2.1 (IN), U2.3 (EN), U3.21 (VCC)
- new net RESET: J9.4
- no-connect marks 0 -> 8
Other:
- note added: "Transient Voltage Supression"
- note added: "pogo pins: usb d+/- 1.8V"
- note removed: "pogo pins: usb d+/- 1.8V GND"
- moved on the sheet: C13, C22, C23, C4, C7, D1, D10, D11, D12, D13, D14, D15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

Commit message: latest iteration with smaller filters and bigger more secure footprint
Parts:
- removed C15, C17, C18, C19, C20, C21, C? (x4): 0.1μF, AU:R_0201_0603Metric, symbol Device:C_Small
- removed D1, D12, D13, D14, D15, D16, D17, D3, D4: TVS, AU:R_0201_0603Metric, symbol Device:D_Zener_Small
- removed D6, D7, D8, D9: 3VWM, AU:R_0201_0603Metric, symbol Device:D_Zener_Small
- removed J10, J11: Conn_02x08_Odd_Even, symbol Connector_Generic:Conn_02x08_Odd_Even
- removed Q?: PFET, AU:CSD23280F3, symbol AU:CSD23280F3
- removed R10, R12, R14, R16, R20, R4: 24, Resistor_SMD:R_0201_0603Metric, symbol Device:R_Small
- removed R11, R13, R15, R17, R21: 51, Resistor_SMD:R_0201_0603Metric, symbol Device:R_Small
- removed R24, R25, R26, R27, R28, R29, R? (x5): 4.7k, Resistor_SMD:R_0201_0603Metric, symbol Device:R_Small
- removed U3: TCA9555RGER, Package_DFN_QFN:VQFN-24-1EP_4x4mm_P0.5mm_EP2.45x2.45mm, symbol Interface_Expansion:TCA9555RGER
- removed U4, U5, U6, U7: TS3DS10224RUK, Package_DFN_QFN:WQFN-20-1EP_3x3mm_P0.4mm_EP1.7x1.7mm, symbol Analog_Switch:TS3DS10224RUK
- added J2: SM04B-SRSS-TB, AU:SM04B-SRSS-TB_JST, symbol AU:SM04B-SRSS-TB
- D2: value TVS -> 2VWM; Alt PN (none) -> CD0201-T2.0LC; MPN ESD1V8AE2-TP -> PESD2V0Y1BSFYL; Manufacturer Micro Commercial Co -> Nexperia USA Inc.
- J1: renamed from J9; footprint AU:CON15_1X15_DRB_SFW_GLE -> AU:528061510
- R1: renamed from R2; footprint Resistor_SMD:R_0201_0603Metric -> AU:R_0201_0603Metric
- R2: renamed from R3; footprint Resistor_SMD:R_0201_0603Metric -> AU:R_0201_0603Metric
- R3: renamed from R7; footprint Resistor_SMD:R_0201_0603Metric -> AU:R_0201_0603Metric
- R4: renamed from R9; footprint Resistor_SMD:R_0201_0603Metric -> AU:R_0201_0603Metric
- R5: value 51 -> 4.7k; footprint Resistor_SMD:R_0201_0603Metric -> AU:R_0201_0603Metric; MPN RMCF0201FT51R0 -> CR0201-JW-472GLF; Manufacturer Stackpole Electronics Inc -> Bourns Inc.; Stock on hand (none) -> 10k; Tolerance 1% -> 5%
- R6: footprint Resistor_SMD:R_0201_0603Metric -> AU:R_0201_0603Metric
- R7: renamed from R1; footprint Resistor_SMD:R_0201_0603Metric -> AU:R_0201_0603Metric
- renumbered C12 to C10, C14 to C11, C16 to C12, C22 to C14, C23 to C15, C4 to C16, C7 to C17, C5 to C4, C6 to C5, C8 to C6, C9 to C7, C10 to C8, C11 to C9, D5 to D1, D10 to D3, D11 to D4, D18 to D5, R18 to R10, R19 to R11, R23 to R8, R8 to R9
Connections:
- net 3V3 is gone; now on net +3V3: C14.2, J1.1, U2.1 (IN), U2.3 (EN)
- net RESET is gone; now on net LED_EN: J1.4
- net +1V8: now also D2.1 (K)
- net CLK-: no longer D2.1 (K)
- net GND: now also J2.2, J2.3, J2.MP; no longer R5.1
- net PWR_EN: now also R5.2; no longer U1.28 (*RESET)
- net video_in1: now also J2.1
- net video_in2: now also J2.4
- net INTRQ: no longer names the net of U1.5 (*INTRQ)
- net video3: no longer names the net of U1.22 (AIN3)
- net video4: no longer names the net of U1.23 (AIN4)
- net video5: no longer names the net of U1.24 (AIN5)
- net video6: no longer names the net of U1.25 (AIN6)
- net video7: no longer names the net of U1.26 (AIN7)
- net video8: no longer names the net of U1.27 (AIN8)
- new net: R5.1, U1.28 (*RESET)
- no-connect marks 8 -> 10
Other:
- note removed: "pogo pins: usb d+/- 1.8V"
- moved on the sheet: D1, D3, D4, D5, R10, R11, R9
